File: GPS Logger/GPSLogger.sch (KiCad schematic (older format))
At the start: 21 parts, among them U1 HM-11, U2 BLE_module, U3 Teensy3.6, U4 GY-91, U5 BME280

Commit message: updated.  needs updates
Parts:
- removed BLE_PWR_Switch1: BLE_PWR_Switch, EbayParts:Pin_Header_1x03_Pitch2.54mm, symbol CONN_01X03
- removed Batt+1: +Batt, EbayParts:Pin_Header_1x01_Pitch2.54mm, symbol CONN_01X01
- removed Batt-1: -Batt, EbayParts:Pin_Header_1x01_Pitch2.54mm, symbol CONN_01X01
- removed BattSwitch1: BattSwitch, EbayParts:Pin_Header_1x03_Pitch2.54mm, symbol CONN_01X03
- removed C1: 82nF, Capacitors_SMD:C_0805_HandSoldering, symbol C
- removed C2: 2.2uF, Capacitors_SMD:C_0805_HandSoldering, symbol C
- removed D1: D, Diodes_SMD:D_SOD-323, symbol D
- removed GPS_CONN1: GPS Connector, EbayParts:Pin_Header_Angled_1x07_Pitch2.54mm, symbol 7pinheader
- removed MAX1: MAX8211, EbayParts:SOIC-8-N, symbol MAX8212
- removed PwrEnFET1: Si6943DQ, EbayParts:TSSOP-8_4.4x3mm_Pitch0.65mm_custom, symbol Si6943DQ
- removed R1, R4, R5: 100k, Resistors_SMD:R_0805_HandSoldering, symbol R_Small
- removed R2: 56k, Resistors_SMD:R_0805_HandSoldering, symbol R_Small
- removed R3: 1M, Resistors_SMD:R_0805_HandSoldering, symbol R_Small
- removed U1: HM-11, EbayParts:HM-11_Breakout, symbol HM-11
- removed U2: BLE_module, EbayParts:HM-10_breakout, symbol BLE_module
- removed U3: Teensy3.6, CustomFP:Teensy35_36, symbol Teensy3.6
- removed U4: GY-91, EbayParts:GY-91, symbol GY-91
- removed U5: BME280, EbayParts:BME280_tiny, symbol BME280
- removed debug_conn1: debug_conn, Pin_Headers:Pin_Header_Angled_1x03_Pitch2.54mm, symbol CONN_01X03
- added C1: 82n, CustomFP:CAM_M8N_V1, symbol Device:C
- added C2: 2.2u, Capacitors_SMD:C_0805, symbol Device:C
- added J1: debug_conn, Connectors2:1X03, symbol Connector:Conn_01x03_Male
- added J2: BLE_Module, EbayParts:HM-10_breakout, symbol Connector:Conn_01x06_Male
- added J3: BLE_PWR_Switch, Connectors2:1X03, symbol Connector:Conn_01x03_Male
- added J4: Conn_01x08_Male, Connectors2:1X08, symbol Connector:Conn_01x08_Male
- added U1: CAM_M8Q, CustomFP:CAM-M8Q, symbol CustomComponents:CAM_M8Q
- added U2: Teensy3.6, CustomFP:Teensy35_36, symbol teensy:Teensy3.6
- added U3: GY-91, EbayParts:GY-91, symbol EbayParts:GY-91
- added U4: BME280, Connectors2:1X04, symbol EbayParts:BME280
Connections:
- net +3V3: now also C1.1, C2.1, J4.2 (Pin_2), U2.15 (3.3V), U2.51 (3.3V_max250mA)
- net BLE_Pwr: now also J2.2 (Pin_2), J3.2 (Pin_2)
- net Fun_Btn_1_P23: now also U2.50 (23_A9_PWM_Touch)
- net Fun_Btn_2_P22: now also U2.49 (22_A8_PWM_Touch)
- net Fun_Btn_3_P21: now also U2.48 (21_A7_PWM_CS0_sck1)
- net GPS_Pwr: now also U1.1 (VCC), U1.9 (VCC)
- net GPS_Pwr_En_P28: now also U2.20 (28)
- net LED1_P2: now also U2.4 (2_PWM)
- net LED2_P3: now also U2.5 (3_PWM_CAN0TX_SCL2)
- net LED3_P4: now also U2.6 (4_PWM_CAN0RX_SDA2)
- net LED4_P5: now also U2.7 (5_PWM_tx1_miso1)
- net Screen_BUSY_P7: now also J4.8 (Pin_8), U2.9 (7_RX3_miso0_scl0)
- net Screen_DC_P8: now also J4.6 (Pin_6), U2.10 (8_TX3_miso0_sda0)
- net Screen_RST_P6: now also J4.7 (Pin_7), U2.8 (6_PWM)
- net Screen_SCK_P27: now also J4.4 (Pin_4), U2.19 (27_rx1)
- net Sensor_PWR_P25: now also U2.17 (25), U3.2 (3V3), U4.1 (Vin)
- net WAKE_UP_PIN: now also U2.18 (26_tx1)
- new net: U1.16 (RF_OUT), U1.17 (RF_IN)
- new net BAttPwr: U2.53 (Vin)
- new net BLE_Rx_TX2_P10: J2.5 (Pin_5), U2.12 (10_PWM_TX2_CS0)
- new net BLE_Tx_RX2_P9: J2.4 (Pin_4), U2.11 (9_PWM_RX2_CS0)
- new net BattPwr: J3.1 (Pin_1)
- new net Debug_Rx_TX5_P33: J1.3 (Pin_3), U2.30 (33_A14_CAN1TX_scl0)
- new net Debug_Tx_RX5_P34: J1.2 (Pin_2), U2.31 (34_A15_CAN1TX_sda0)
- new net GNDREF: C1.2, C2.2, J1.1 (Pin_1), J2.3 (Pin_3), J4.1 (Pin_1), U1.10 (GND), U1.11 (GND), U1.12 (GND), U1.13 (GND), U1.14 (GND), U1.15 (GND), U1.18 (GND), U1.19 (GND), U1.21 (GND), U1.22 (GND), U1.27 (GND), U1.31 (GND), U1.4 (GND), U1.5 (GND), U2.1 (GND), U2.39 (GND), U3.3 (GND), U3.6 (SDO), U3.8 (CSB), U4.2 (GND)
- new net GPS_ExtInt_P37: U1.7 (EXTINT), U2.34 (37_A18_PWM_SCL1)
- new net GPS_Reset_P39: U1.23 (RESET_N), U2.36 (39_A20)
- new net GPS_Rx_TX1_P1: U1.26 (RXD), U2.3 (1_TX1_MISO1_Touch)
- new net GPS_TimePulse_P38: U1.29 (TimePulse), U2.35 (38_A19_PWM_SDA1)
- new net GPS_Tx_RX1_P0: U1.25 (TXD), U2.2 (0_RX1_MOSI1_Touch)
- new net SCL: U2.46 (19_A5_SCL0_Touch), U3.4 (SCL), U4.3 (SCL)
- new net SDA: U2.45 (18_A4_SDA0_Touch), U3.5 (SDA), U4.4 (SDA)
- new net Screen_CS_P20: J4.5 (Pin_5), U2.47 (20_A6_PWM_CS0_sck1)
- new net Screen_DIN_P11: J4.3 (Pin_3), U2.13 (11_MOSI0)
- new net USBPwr: U2.54 (VUSB)
- no-connect marks 72 -> 60
