File: GPS Logger/GPSLogger.kicad_pcb (KiCad board)
At the start: 2 copper layers, 101.9 x 77.5 mm, 43 parts, among them U1 HM-11, U3 Teensy3.6, U4 GY-91, U5 BME280, U6 APM4953, U7 APM4953

Commit message: updated.  needs updates
Parts:
- removed BLE_PWR_Switch1: BLE_PWR_Switch, EbayParts:Pin_Header_1x03_Pitch2.54mm
- removed Batt+1: +Batt, EbayParts:Pin_Header_1x01_Pitch2.54mm
- removed Batt-1: -Batt, EbayParts:Pin_Header_1x01_Pitch2.54mm
- removed BattSwitch1: BattSwitch, EbayParts:Pin_Header_1x03_Pitch2.54mm
- removed Fun_BTN1: Fun_BTN, EbayParts:SMD_Switch_3x6
- removed Fun_BTN2, Fun_BTN3: LVCutoff_reset, EbayParts:SMD_Switch_3x6
- removed GPS_CONN1: GPS Connector, EbayParts:Pin_Header_Angled_1x07_Pitch2.54mm
- removed LED_D1: BLUE, LEDs:LED_0805
- removed LED_D2: GREEN, LEDs:LED_0805
- removed LED_D3: RED, LEDs:LED_0805
- removed LED_D4: ORANGE, LEDs:LED_0805
- removed LED_R1: 5.6, Resistors_SMD:R_0805_HandSoldering
- removed LED_R2: 10, Resistors_SMD:R_0805_HandSoldering
- removed LED_R3, LED_R4: 56, Resistors_SMD:R_0805_HandSoldering
- removed MAX1: MAX8211, EbayParts:SOIC-8-N
- removed PwrEnFET1: Si6943DQ, EbayParts:TSSOP-8_4.4x3mm_Pitch0.65mm_custom
- removed REF**: CAM_M8N_V1, CustomFP:CAM_M8N_V1
- removed REF**: EInk_154in, CustomFP:EInk_154in
- removed STS_LED_EN1: STS_LED_EN, EbayParts:SMD_Switch_3x6
- removed debug_conn1: debug_conn, Pin_Headers:Pin_Header_Angled_1x03_Pitch2.54mm
- added C3: 0.1u, Capacitors_SMD:C_0805, F.Cu at (247.5, 36.5)
- added C4: 1u, Capacitors_SMD:C_0805, F.Cu at (192.5, 46.2)
- added C5: 2.2u, Capacitors_SMD:C_0805, F.Cu at (234.0, 36.5)
- added C6: 0.1u, Capacitors_SMD:C_0805, F.Cu at (201.8, 37.9)
- added D2: LED_G, LEDs:LED_0805, F.Cu at (93.0, 101.5)
- added D3: LED_R, LEDs:LED_0805, F.Cu at (55.9, 92.5)
- added D4: LED_O, LEDs:LED_0805, F.Cu at (55.1, 111.5)
- added D5: LED, LEDs:LED_0805, F.Cu at (243.5, 47.0)
- added J1: debug_conn, Connectors2:1X03, F.Cu at (154.8, 43.9)
- added J10: Batt+, Connectors2:1X01, F.Cu at (214.5, 64.0)
- added J11: Batt-, Connectors2:1X01, F.Cu at (195.5, 60.0)
- added J2: BLE_Module, EbayParts:HM-10_breakout, F.Cu at (112.9, 87.1)
- added J3: BLE_PWR_Switch, Connectors2:1X03, F.Cu at (154.0, 56.3)
- added J4: Conn_01x08_Male, Connectors2:1X08, F.Cu at (80.0, 74.3)
- added J5: LED_BUTTON, EbayParts:Tact_SMD_Switch, F.Cu at (77.0, 102.0)
- added J6: BTN1, EbayParts:Tact_SMD_Switch, F.Cu at (98.7, 94.8)
- added J7: BTN1, EbayParts:Tact_SMD_Switch, F.Cu at (86.5, 117.0)
- added J8: BTN1, EbayParts:Tact_SMD_Switch, F.Cu at (105.7, 94.8)
- added J9: Battery Switch, Connectors2:1X03, F.Cu at (187.3, 38.4)
- added JP1: Jumper_NO_Small, Jumpers:SMT-JUMPER_2_NO_NO-SILK, F.Cu at (226.1, 56.1)
- added JP2: Jumper_NC_Small, Jumpers:SMT-JUMPER_2_NC_PASTE_SILK, F.Cu at (204.6, 46.5)
- added R13: 330, Resistors_SMD:R_0805, F.Cu at (216.0, 28.0)
- added R14: 100, Resistors_SMD:R_0805, F.Cu at (221.6, 50.5)
- added R15: 100, Resistors_SMD:R_0805, F.Cu at (201.4, 56.0)
- added R16: 10, Resistors_SMD:R_0805, F.Cu at (243.0, 56.5)
- added R17: 10M, Resistors_SMD:R_0805, F.Cu at (205.3, 41.7)
- added R18: 10M, Resistors_SMD:R_0805, F.Cu at (209.6, 33.0)
- added TH1: NTC, Resistors_SMD:R_0805, F.Cu at (205.4, 65.0)
- added TH2: NTC, Resistors_SMD:R_0805, F.Cu at (234.4, 62.5)
- added U2: Teensy3.6, CustomFP:Teensy35_36, F.Cu at (112.5, 44.5)
- added U8: CEM9926A, EbayParts:SOIC-8-N, F.Cu at (178.5, 29.5)
- C1: value 82nF -> 82n; footprint Capacitors_SMD:C_0805_HandSoldering -> CustomFP:CAM_M8N_V1
- C2: value 2.2uF -> 2.2u; footprint Capacitors_SMD:C_0805_HandSoldering -> Capacitors_SMD:C_0805
- D1: value D -> LED_B; footprint Diodes_SMD:D_SOD-323 -> LEDs:LED_0805; moved to F.Cu
- R1: value 100k -> 10k; footprint Resistors_SMD:R_0805_HandSoldering -> Resistors_SMD:R_0805; moved to F.Cu
- R10, R12: value 10k -> 100; footprint Resistors_SMD:R_0805_HandSoldering -> Resistors_SMD:R_0805; moved to F.Cu
- R11: value 10k -> 1m; footprint Resistors_SMD:R_0805_HandSoldering -> Resistors_SMD:R_0805; moved to F.Cu
- R2: value 56k -> 5.6; footprint Resistors_SMD:R_0805_HandSoldering -> Resistors_SMD:R_0805; moved to F.Cu
- R3: value 1M -> 10; footprint Resistors_SMD:R_0805_HandSoldering -> Resistors_SMD:R_0805; moved to F.Cu
- R4: value 100k -> 56; footprint Resistors_SMD:R_0805_HandSoldering -> Resistors_SMD:R_0805
- R5: value 100k -> 56; footprint Resistors_SMD:R_0805_HandSoldering -> Resistors_SMD:R_0805; moved to F.Cu
- R6, R7, R8: footprint Resistors_SMD:R_0805_HandSoldering -> Resistors_SMD:R_0805
- R9: value 100k -> Riset; footprint Resistors_SMD:R_0805_HandSoldering -> Resistors_SMD:R_0805
- U1: value HM-11 -> CAM_M8Q; footprint EbayParts:HM-11 -> CustomFP:CAM-M8Q; moved to F.Cu
- U3: value Teensy3.6 -> GY-91; footprint CustomFP:Teensy35_36 -> EbayParts:GY-91
- U4: value GY-91 -> BME280; footprint EbayParts:GY-91 -> Connectors2:1X04; moved to F.Cu
- U5: value BME280 -> APM4953; footprint EbayParts:BME280_tiny -> EbayParts:SOIC-8-N; moved to F.Cu
- U6: value APM4953 -> BQ21040; footprint Housings_SOIC:SOIC-8_3.9x4.9mm_Pitch1.27mm -> CustomFP:BQ21040
- U7: value APM4953 -> BQ27750; footprint Housings_SOIC:SOIC-8_3.9x4.9mm_Pitch1.27mm -> CustomFP:BQ27750
- moved R10 155.0 mm to (229.7, 50.8), turned to 0 degrees
- moved R11 140.4 mm to (215.5, 56.0), turned to 0 degrees
- moved U4 131.6 mm to (154.8, 41.1), turned to 0 degrees
- moved R12 108.3 mm to (192.3, 54.0), turned to 0 degrees
- moved R7 106.8 mm to (68.5, 118.5)
- moved R6 104.8 mm to (57.1, 103.6)
- moved U1 81.9 mm to (58.4, 48.6), turned to 0 degrees
- moved C1 69.0 mm to (122.0, 85.5)
- moved U7 66.0 mm to (199.0, 31.0)
- moved R9 64.5 mm to (215.5, 39.5)
- moved R5 64.1 mm to (79.0, 110.5), turned to 0 degrees
- moved R8 59.7 mm to (106.6, 97.8)
- moved U3 52.1 mm to (154.8, 38.4), turned to 0 degrees
- moved R3 49.9 mm to (109.7, 97.9), turned to 0 degrees
- moved R4 49.3 mm to (109.7, 96.0)
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Connections:
- C2 pad 2: GND -> BattRtn
- D1 pad 1: /BattPostSwitch -> Net-(D1-Pad1)
- D1 pad 2: /USBPower+ -> LED1_P2
- R1 pad 1: Net-(MAX1-Pad3) -> Net-(R1-Pad1)
- R1 pad 2: +BATT -> (no net)
- R10 pad 1: Fun_Btn_3_P21 -> Net-(C3-Pad2)
- R10 pad 2: GND -> BattRtn
- R11 pad 1: Fun_Btn_2_P22 -> Net-(C4-Pad2)
- R11 pad 2: GND -> BattRtn
- R12 pad 1: Fun_Btn_1_P23 -> Net-(C3-Pad1)
- R12 pad 2: GND -> Net-(C4-Pad2)
- R2 pad 1: GND -> Net-(D1-Pad1)
- R2 pad 2: Net-(MAX1-Pad3) -> Net-(J5-Pad2)
- R3 pad 2: /BattPostSwitch -> Net-(J5-Pad2)
- R4 pad 1: GND -> Net-(D3-Pad1)
- R4 pad 2: (no net) -> Net-(J5-Pad2)
- R5 pad 1: GND -> Net-(D4-Pad1)
- R5 pad 2: /USBPower+ -> Net-(J5-Pad2)
- R6 pad 1: Net-(R6-Pad1) -> Fun_Btn_1_P23
- R6 pad 2: GPS_Pwr_En_P7 -> BattRtn
- R7 pad 1: Net-(R7-Pad1) -> Fun_Btn_2_P22
- R7 pad 2: Batt_Mon_En_P20 -> BattRtn
- R8 pad 1: Net-(R8-Pad1) -> Fun_Btn_3_P21
- R8 pad 2: Batt_Mon_P35 -> BattRtn
- R9 pad 1: Batt_Mon_P35 -> BattRtn
- R9 pad 2: GND -> Net-(R9-Pad2)
- U1 pad 1: Net-(U1-Pad1) -> GPS_Pwr
- U1 pad 10: (no net) -> BattRtn
- U1 pad 11: Net-(U1-Pad11) -> BattRtn
- U1 pad 12: Net-(U1-Pad12) -> BattRtn
- U1 pad 13: Net-(U1-Pad13) -> BattRtn
- U1 pad 14: Net-(U1-Pad14) -> BattRtn
- U1 pad 15: Net-(U1-Pad15) -> BattRtn
- U1 pad 2: Net-(U1-Pad2) -> (no net)
- U1 pad 3: Net-(U1-Pad3) -> (no net)
- U1 pad 4: Net-(U1-Pad4) -> BattRtn
- U1 pad 5: Net-(U1-Pad5) -> BattRtn
- U1 pad 6: Net-(U1-Pad6) -> (no net)
- U1 pad 7: Net-(U1-Pad7) -> (no net)
- U1 pad 9: Net-(U1-Pad9) -> GPS_Pwr
- U3 pad 1: GND -> (no net)
- U3 pad 2: /Debug_Rx_TX1_P0 -> /Sensor_PWR_P25
- U3 pad 3: /Debug_Tx_RX1_P1 -> BattRtn
- U3 pad 4: LED1_P2 -> SCL
- U3 pad 5: LED2_P3 -> SDA
- U3 pad 6: LED3_P4 -> BattRtn
- U3 pad 7: LED4_P5 -> (no net)
- U3 pad 8: (no net) -> BattRtn
- U4 pad 1: +3V3 -> /Sensor_PWR_P25
- U4 pad 2: (no net) -> BattRtn
- U4 pad 3: GND -> SCL
- U4 pad 4: /I2c_SCL_P19 -> SDA
- U5 pad 2: GND -> Net-(R1-Pad1)
- U5 pad 3: /I2c_SCL_P19 -> +3V3
- U5 pad 4: /I2c_SDA_P18 -> Net-(R1-Pad1)
- U6 pad 1: +3V3 -> USBPwr
- U6 pad 2: Net-(R6-Pad1) -> Net-(R9-Pad2)
- U6 pad 3: +3V3 -> BattRtn
- U6 pad 4: Net-(R6-Pad1) -> Net-(TH1-Pad1)
- U6 pad 5: GPS_Pwr -> Net-(D5-Pad1)
- U6 pad 6: GPS_Pwr -> Net-(C4-Pad1)
- U7 pad 1: +BATT -> Net-(C4-Pad2)
- U7 pad 2: Net-(R7-Pad1) -> Net-(C3-Pad2)
- U7 pad 3: +BATT -> Net-(C3-Pad1)
- U7 pad 4: Net-(R7-Pad1) -> Net-(TH2-Pad1)
- U7 pad 5: Net-(R8-Pad1) -> Net-(R14-Pad1)
- U7 pad 6: Net-(R8-Pad1) -> Net-(R15-Pad1)
- U7 pad 7: Net-(R8-Pad1) -> Net-(R17-Pad1)
- U7 pad 8: Net-(R8-Pad1) -> Net-(R16-Pad1)
Other:
- board outline removed
- net class Default: clearance 0.254 -> 0.2; trace_width 0.254 -> 0.25; via_dia 0.381 -> 0.8; via_drill 0.254 -> 0.4
- rule trace_clearance: 0.254 -> 0.2
- rule trace_min: 0.1524 -> 0.2
- rule via_min_drill: 0.254 -> 0.3
- rule via_min_size: 0.381 -> 0.4
- board text removed: "Off"
- board text removed: "On"
- board text removed: "Scott Co. GPS Logger V4"
- board text removed: "Tx Rx"

Commit message: Orders from JLCPCB
Parts:
- removed C1: 82n, CustomFP:CAM_M8N_V1
- removed J11: Batt-, Connectors2:1X01
- removed R11: 1m, Resistors_SMD:R_0805
- removed R14, R15: 100, Resistors_SMD:R_0805
- added JP3: Jumper_NO_Small, Jumpers:SMT-JUMPER_2_NO_NO-SILK, B.Cu at (158.9, 75.0)
- added JP4: Jumper_NO_Small, Jumpers:SMT-JUMPER_2_NO_NO-SILK, B.Cu at (160.9, 75.0)
- added U9: R_0612, Resistor_SMD:R_Shunt_Vishay_WSKW0612, F.Cu at (158.3, 70.4)
- C5, J2, R16, R18, R2, R3, R4, R5, R6, R7, R8, TH2, U2, U8: moved to B.Cu
- J10: value Batt+ -> Conn_01x03_Male; footprint Connectors2:1X01 -> CustomFP:molex_78172-0003; moved to B.Cu
- J7: value BTN1 -> BTN2
- J8: value BTN1 -> BTN3
- moved U1 112.2 mm to (160.5, 95.0), turned to 180 degrees
- moved U5 111.5 mm to (151.5, 72.1), turned to 180 degrees
- moved C3 100.1 mm to (156.1, 77.2)
- moved R6 94.6 mm to (148.8, 80.2)
- moved D3 91.2 mm to (147.1, 89.9)
- moved D4 90.3 mm to (142.7, 89.9)
- moved R7 90.0 mm to (148.8, 77.8)
- moved D1 89.7 mm to (147.1, 92.8)
- moved D5 87.3 mm to (156.3, 44.2), turned to 90 degrees
- moved J4 84.5 mm to (153.4, 32.5), turned to 270 degrees
- moved R16 84.5 mm to (158.8, 62.4), turned to 270 degrees
- moved C5 80.7 mm to (155.3, 54.7), turned to 90 degrees
- moved J2 76.3 mm to (161.0, 27.9), turned to 90 degrees
- moved TH2 76.1 mm to (159.9, 77.5), turned to 180 degrees
- moved R10 73.8 mm to (160.1, 75.5), turned to 90 degrees
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Connections:
- J10 pad 1: Net-(J10-Pad1) -> Net-(C4-Pad2)
- J9 pad 1: Net-(J10-Pad1) -> Net-(J10-Pad3)
- R1 pad 2: (no net) -> GPS_Pwr_En_P28
- R10 pad 2: BattRtn -> Net-(R10-Pad2)
- R12 pad 2: Net-(C4-Pad2) -> Net-(R12-Pad2)
- TH2 pad 1: Net-(TH2-Pad1) -> Net-(JP4-Pad2)
- U2 pad 53: (no net) -> BattPwr
- U7 pad 4: Net-(TH2-Pad1) -> Net-(JP3-Pad1)
- U7 pad 5: Net-(R14-Pad1) -> SCL
- U7 pad 6: Net-(R15-Pad1) -> SDA
Routing:
- net BattRtn: track 0.00 -> 235.8 mm, vias 0 -> 4
- net +3V3: track 0.00 -> 108.5 mm, vias 0 -> 4
- net BattPwr: track 0.00 -> 71.9 mm
- net Net-(C4-Pad2): track 0.00 -> 67.9 mm, vias 0 -> 5
- net GPS_Pwr_En_P28: track 0.00 -> 64.4 mm, vias 0 -> 4
- net Net-(C4-Pad1): track 0.00 -> 58.6 mm, vias 0 -> 3
- net SDA: track 0.00 -> 55.9 mm
- net USBPwr: track 0.00 -> 55.2 mm
- net SCL: track 0.00 -> 50.8 mm
- net /BLE_Tx_RX2_P9: track 0.00 -> 43.6 mm, vias 0 -> 1
- net /BLE_Rx_TX2_P10: track 0.00 -> 41.6 mm, vias 0 -> 1
- net /Screen_BUSY_P7: track 0.00 -> 38.4 mm
- net Net-(C3-Pad2): track 0.00 -> 37.7 mm, vias 0 -> 2
- net /Screen_CS_P20: track 0.00 -> 36.2 mm, vias 0 -> 2
- net /GPS_Rx_TX1_P1: track 0.00 -> 34.2 mm, vias 0 -> 2
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- added copper zone on B.Cu, net BattRtn
- added copper zone on F.Cu, net BattRtn
Other:
- board outline added: 34.5 x 69 mm
- net class Default: clearance 0.2 -> 0.15
- net class small added: clearance 0.15, trace_width 0.125, via_dia 0.8, via_drill 0.4
- rule trace_clearance: 0.2 -> 0.15
- rule trace_min: 0.2 -> 0.0889
- rule via_min_drill: 0.3 -> 0.2
- rule via_min_size: 0.4 -> 0.45
