File: GPS Logger/file5AC349CC.sch (KiCad schematic (older format))
At the start: 23 parts, among them U6 APM4953, U7 APM4953

Commit message: updated.  needs updates
Parts:
- removed Fun_BTN1: Fun_BTN, EbayParts:SMD_Switch_3x6, symbol CONN_01X02
- removed Fun_BTN2, Fun_BTN3: LVCutoff_reset, EbayParts:SMD_Switch_3x6, symbol CONN_01X02
- removed LED_D1: BLUE, LEDs:LED_0805, symbol LED
- removed LED_D2: GREEN, LEDs:LED_0805, symbol LED
- removed LED_D3: RED, LEDs:LED_0805, symbol LED
- removed LED_D4: ORANGE, LEDs:LED_0805, symbol LED
- removed LED_R1: 5.6, Resistors_SMD:R_0805_HandSoldering, symbol R_Small
- removed LED_R2: 10, Resistors_SMD:R_0805_HandSoldering, symbol R_Small
- removed LED_R3, LED_R4: 56, Resistors_SMD:R_0805_HandSoldering, symbol R_Small
- removed R10, R11, R12, R6, R7, R8, R?: 10k, Resistors_SMD:R_0805_HandSoldering, symbol R_Small
- removed R9: 100k, Resistors_SMD:R_0805_HandSoldering, symbol R_Small
- removed STS_LED_EN1: STS_LED_EN, EbayParts:SMD_Switch_3x6, symbol CONN_01X02
- removed U6, U7: APM4953, Housings_SOIC:SOIC-8_3.9x4.9mm_Pitch1.27mm, symbol APM4953
- removed U?: NPN_3904, symbol NPN_3904
- added D1: LED_B, LEDs:LED_0805, symbol Device:LED
- added D2: LED_G, LEDs:LED_0805, symbol Device:LED
- added D3: LED_R, LEDs:LED_0805, symbol Device:LED
- added D4: LED_O, LEDs:LED_0805, symbol Device:LED
- added J5: LED_BUTTON, EbayParts:Tact_SMD_Switch, symbol Connector:Conn_01x02_Male
- added J6, J7, J8: BTN1, EbayParts:Tact_SMD_Switch, symbol Connector:Conn_01x02_Male
- added R1, R6, R7, R8: 10k, Resistors_SMD:R_0805, symbol Device:R
- added R2: 5.6, Resistors_SMD:R_0805, symbol Device:R
- added R3: 10, Resistors_SMD:R_0805, symbol Device:R
- added R4, R5: 56, Resistors_SMD:R_0805, symbol Device:R
- added U5: APM4953, EbayParts:SOIC-8-N, symbol EbayParts:APM4953
Connections:
- net labels added: BattRtn, GNDREF
- net labels removed: +BATT, Batt_Mon_En_P20, Batt_Mon_P35, GNDPWR
- wire segments 31 -> 25

Commit message: Orders from JLCPCB
Parts:
- J7: value BTN1 -> BTN2
- J8: value BTN1 -> BTN3
- U5: symbol EbayParts:APM4953 -> GPSLogger-rescue:APM4953-EbayParts
Changed lines of the file:
@@
 $EndComp
 $Comp
-L EbayParts:APM4953 U5
+L GPSLogger-rescue:APM4953-EbayParts U5
 U 1 1 5BC171BF
 P 5500 2250
+AR Path="/5BC171BF" Ref="U5"  Part="1"
+AR Path="/5AC349CD/5BC171BF" Ref="U5"  Part="1"
 F 0 "U5" H 5750 2697 60  0000 C CNN
 F 1 "APM4953" H 5750 2591 60  0000 C CNN
@@
 P 8850 2350
 F 0 "J7" H 8823 2230 50  0000 R CNN
-F 1 "BTN1" H 8823 2321 50  0000 R CNN
+F 1 "BTN2" H 8823 2321 50  0000 R CNN
 F 2 "EbayParts:Tact_SMD_Switch" H 8850 2350 50  0001 C CNN
 F 3 "~" H 8850 2350 50  0001 C CNN
@@
 P 8850 3250
 F 0 "J8" H 8823 3130 50  0000 R CNN
-F 1 "BTN1" H 8823 3221 50  0000 R CNN
+F 1 "BTN3" H 8823 3221 50  0000 R CNN
 F 2 "EbayParts:Tact_SMD_Switch" H 8850 3250 50  0001 C CNN
 F 3 "~" H 8850 3250 50  0001 C CNN
