File: GPS Logger/BMS.sch (KiCad schematic (older format))
At the start: 25 parts, among them J10 Batt+, J11 Batt-, J9 Battery Switch, U6 BQ21040, U7 BQ27750, U8 CEM9926A

Commit message: Orders from JLCPCB
Parts:
- removed J10: Batt+, Connectors2:1X01, symbol Connector:Conn_01x01_Male
- removed J11: Batt-, Connectors2:1X01, symbol Connector:Conn_01x01_Male
- removed R11: 1m, Resistors_SMD:R_0805, symbol Device:R
- removed R14, R15: 100, Resistors_SMD:R_0805, symbol Device:R
- added J10: Conn_01x03_Male, CustomFP:molex_78172-0003, symbol Connector:Conn_01x03_Male
- added JP3, JP4: Jumper_NO_Small, Jumpers:SMT-JUMPER_2_NO_NO-SILK, symbol Device:Jumper_NO_Small
- added U9: R_0612, Resistor_SMD:R_Shunt_Vishay_WSKW0612, symbol CustomComponents:R_0612
Connections:
- wire segments 73 -> 86
Other:
- moved on the sheet: TH2
Changed lines of the file:
@@
 	8200 3300 8350 3300
 Wire Wire Line
-	7600 3600 7600 3650
-Wire Wire Line
-	7300 3650 7300 3600
-Wire Wire Line
 	7600 3300 7600 3100
 Wire Wire Line
@@
 	7300 3000 7300 3300
 Wire Wire Line
-	7950 3550 7950 3650
-Connection ~ 7950 3650
-Wire Wire Line
-	7950 3250 7950 3200
-Wire Wire Line
-	7950 3200 8350 3200
-Wire Wire Line
 	8350 2900 8150 2900
 Wire Wire Line
 	8150 2600 8150 2900
-Connection ~ 8150 3650
 Wire Wire Line
 	8300 4400 7900 4400
-Wire Wire Line
-	7600 3650 7950 3650
 Wire Wire Line
 	6150 3650 7100 3650
@@
 Wire Wire Line
 	7100 2700 7100 3650
-Connection ~ 7100 3650
 Wire Wire Line
 	7000 2150 7300 2150
@@
 Text GLabel 6150 3650 0    60   Input ~ 0
 BattRtn
-Text GLabel 7600 4250 0    60   Input ~ 0
+Text GLabel 7900 4250 0    60   Input ~ 0
 SCL
-Text GLabel 7600 4400 0    60   Input ~ 0
+Text GLabel 7900 4400 0    60   Input ~ 0
 SDA
-Wire Wire Line
-	7950 3650 8150 3650
-Wire Wire Line
-	7100 3650 7300 3650
 Wire Wire Line
 	6150 2450 6150 2250
@@
 Connection ~ 7000 2050
 Wire Wire Line
-	8850 3650 10200 3650
+	8850 3650 9550 3650
 $Comp
 L Device:R R17
@@
 $EndComp
 $Comp
-L Connector:Conn_01x01_Male J10
-U 1 1 5BB9DD63
-P 10700 3000
-F 0 "J10" H 10673 2930 50  0000 R CNN
-F 1 "Batt+" H 10673 3021 50  0000 R CNN
-F 2 "Connectors2:1X01" H 10700 3000 50  0001 C CNN
-F 3 "~" H 10700 3000 50  0001 C CNN
-	1    10700 3000
-	-1   0    0    1
-$EndComp
-$Comp
-L Connector:Conn_01x01_Male J11
-U 1 1 5BB9DDCC
-P 10850 3650
-F 0 "J11" H 10823 3580 50  0000 R CNN
-F 1 "Batt-" H 10823 3671 50  0000 R CNN
-F 2 "Connectors2:1X01" H 10850 3650 50  0001 C CNN
-F 3 "~" H 10850 3650 50  0001 C CNN
-	1    10850 3650
-	-1   0    0    1
-$EndComp
-$Comp
 L Device:C C6
 U 1 1 5BB9E29D
@@
 Connection ~ 10400 3650
 Wire Wire Line
-	10400 3650 10650 3650
+	10400 3650 10600 3650
 $Comp
 L Device:C C5
@@
 	10400 2700 10400 2900
 Connection ~ 10400 2900
-Wire Wire Line
-	10500 2800 10500 3000
 $Comp
 L Device:R R16
@@
 L Device:Thermistor_NTC TH2
 U 1 1 5BBA528E
-P 7950 3400
-F 0 "TH2" H 8047 3446 50  0000 L CNN
-F 1 "NTC" H 8047 3355 50  0000 L CNN
-F 2 "Resistors_SMD:R_0805" H 7950 3450 50  0001 C CNN
-F 3 "~" H 7950 3450 50  0001 C CNN
-	1    7950 3400
+P 8850 4100
+F 0 "TH2" H 8947 4146 50  0000 L CNN
+F 1 "NTC" H 8947 4055 50  0000 L CNN
+F 2 "Resistors_SMD:R_0805" H 8850 4150 50  0001 C CNN
+F 3 "~" H 8850 4150 50  0001 C CNN
+	1    8850 4100
 	1    0    0    -1
 $EndComp
@@
 $EndComp
 $Comp
-L Device:R R11
-U 1 1 5BBA5979
-P 7450 3650
-F 0 "R11" V 7243 3650 50  0000 C CNN
-F 1 "1m" V 7334 3650 50  0000 C CNN
-F 2 "Resistors_SMD:R_0805" V 7380 3650 50  0001 C CNN
-F 3 "~" H 7450 3650 50  0001 C CNN
-	1    7450 3650
-	0    1    1    0
-$EndComp
-$Comp
 L Device:R R10
 U 1 1 5BBA5B49
@@
 	0    1    1    0
 $EndComp
-$Comp
-L Device:R R14
-U 1 1 5BBA5F9C
-P 7750 4250
-F 0 "R14" V 7650 4200 50  0000 L CNN
-F 1 "100" V 7750 4200 50  0000 L CNN
-F 2 "Resistors_SMD:R_0805" V 7680 4250 50  0001 C CNN
-F 3 "~" H 7750 4250 50  0001 C CNN
-	1    7750 4250
-	0    1    1    0
-$EndComp
-$Comp
-L Device:R R15
-U 1 1 5BBA603C
-P 7750 4400
-F 0 "R15" V 7850 4350 50  0000 L CNN
-F 1 "100" V 7750 4350 50  0000 L CNN
-F 2 "Resistors_SMD:R_0805" V 7680 4400 50  0001 C CNN
-F 3 "~" H 7750 4400 50  0001 C CNN
-	1    7750 4400
-	0    1    1    0
-$EndComp
 Connection ~ 7300 3300
 Connection ~ 7600 3300
-Connection ~ 7600 3650
-Connection ~ 7300 3650
 $Comp
 L Device:Thermistor_NTC TH1
@@
 Wire Wire Line
 	7900 2050 8150 2050
+$Comp
+L Connector:Conn_01x03_Male J10
+U 1 1 5BF48585
+P 10800 3100
+F 0 "J10" H 10773 3030 50  0000 R CNN
+F 1 "Conn_01x03_Male" H 10773 3121 50  0000 R CNN
+F 2 "CustomFP:molex_78172-0003" H 10800 3100 50  0001 C CNN
+F 3 "~" H 10800 3100 50  0001 C CNN
+	1    10800 3100
+	-1   0    0    1
+$EndComp
+Wire Wire Line
+	10600 3000 10500 3000
+Wire Wire Line
+	10500 3000 10500 2800
+Wire Wire Line
+	10600 3200 10600 3650
+Wire Wire Line
+	10600 3100 10500 3100
+Wire Wire Line
+	10500 3100 10500 3850
+$Comp
+L Device:Jumper_NO_Small JP4
+U 1 1 5BF51354
+P 8750 3950
+F 0 "JP4" H 8750 4135 50  0000 C CNN
+F 1 "Jumper_NO_Small" H 8750 4044 50  0000 C CNN
+F 2 "Jumpers:SMT-JUMPER_2_NO_NO-SILK" H 8750 3950 50  0001 C CNN
+F 3 "~" H 8750 3950 50  0001 C CNN
+	1    8750 3950
+	1    0    0    -1
+$EndComp
+Wire Wire Line
+	8850 4250 9550 4250
+Wire Wire Line
+	9550 4250 9550 3650
+Connection ~ 9550 3650
+Wire Wire Line
+	9550 3650 10200 3650
+$Comp
+L Device:Jumper_NO_Small JP3
+U 1 1 5BF52D7D
+P 8750 3850
+F 0 "JP3" H 8750 4035 50  0000 C CNN
+F 1 "Jumper_NO_Small" H 8750 3944 50  0000 C CNN
+F 2 "Jumpers:SMT-JUMPER_2_NO_NO-SILK" H 8750 3850 50  0001 C CNN
+F 3 "~" H 8750 3850 50  0001 C CNN
+	1    8750 3850
+	1    0    0    -1
+$EndComp
+Wire Wire Line
+	8850 3850 10500 3850
+Wire Wire Line
+	8650 3850 8650 3950
+Wire Wire Line
+	8650 3850 7950 3850
+Wire Wire Line
+	7950 3850 7950 3200
+Wire Wire Line
+	7950 3200 8350 3200
+Connection ~ 8650 3850
+$Comp
+L CustomComponents:R_0612 U9
+U 1 1 5BF27423
+P 7450 3700
+F 0 "U9" H 7450 3485 50  0000 C CNN
+F 1 "R_0612" H 7450 3576 50  0000 C CNN
+F 2 "Resistor_SMD:R_Shunt_Vishay_WSKW0612" H 7450 3700 50  0001 C CNN
+F 3 "" H 7450 3700 50  0001 C CNN
+	1    7450 3700
+	1    0    0    1
+$EndComp
+Wire Wire Line
+	7200 3700 7200 3600
+Wire Wire Line
+	7200 3600 7300 3600
+Wire Wire Line
+	7600 3600 7700 3600
+Wire Wire Line
+	7700 3600 7700 3700
+Wire Wire Line
+	7700 3800 7850 3800
+Wire Wire Line
+	7850 3800 7850 3650
+Wire Wire Line
+	7850 3650 8150 3650
+Connection ~ 8150 3650
+Wire Wire Line
+	7200 3800 7100 3800
+Wire Wire Line
+	7100 3800 7100 3650
+Connection ~ 7100 3650
 $EndSCHEMATC

Commit message: pcb updates
Parts:
- removed JP3, JP4: Jumper_NO_Small, Jumpers:SMT-JUMPER_2_NO_NO-SILK, symbol Device:Jumper_NO_Small
- removed U6: BQ21040, CustomFP:BQ21040, symbol CustomComponents:BQ21040
- added U?: BQ21040, symbol CustomComponents:BQ21040
- R9: value Riset -> 1k
- renumbered U9 to R98
Connections:
- net BattRtn: now also TH1.1, U?.5 (GND); no longer TH1.2
- net USBPwr: now also U?.6 (VIN)
- net at U7.4 (TS1): now also TH2.1
- net at D5.1 (K): now also U?.3 (~CHG)
- net at C4.1, JP1.2, JP2.2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: now also U?.2 (VOUT)
- net at R9.2: now also U?.4 (ISET)
- new net: TH1.2, U?.1 (TS)
- no-connect marks 1 -> 2
Other:
- moved on the sheet: C3, D5, R10, R12, R13, R98, TH1, TH2
Changed lines of the file:
@@
 	9400 3100 10200 3100
 $Bitmap
-Pos 14000 1550
+Pos 13050 2450
 Scale 1.000000
 Data
@@
 	8200 3300 8350 3300
 Wire Wire Line
-	7600 3300 7600 3100
+	7700 3100 8350 3100
 Wire Wire Line
-	7600 3100 8350 3100
-Wire Wire Line
-	8350 3000 7300 3000
-Wire Wire Line
-	7300 3000 7300 3300
+	8350 3000 7200 3000
 Wire Wire Line
 	8350 2900 8150 2900
@@
 Wire Wire Line
 	8300 4400 7900 4400
-Wire Wire Line
-	6150 3650 7100 3650
-Text Notes 7000 2000 0    60   ~ 0
+Text Notes 9000 2050 0    60   ~ 0
 Pack+
-Text Notes 7000 3750 0    60   ~ 0
+Text Notes 6600 3650 0    60   ~ 0
 Pack-
 Wire Wire Line
 	10400 3350 10400 2900
 Wire Wire Line
-	7000 2250 7100 2250
-Wire Wire Line
-	7100 2250 7100 2400
-Wire Wire Line
-	7100 2700 7100 3650
-Wire Wire Line
-	7000 2150 7300 2150
-Wire Wire Line
 	6150 2050 5850 2050
 Wire Wire Line
@@
 Connection ~ 8850 3650
 $Comp
-L CustomComponents:BQ21040 U6
-U 1 1 5BB6F51A
-P 6550 2200
-F 0 "U6" H 6575 2597 60  0000 C CNN
-F 1 "BQ21040" H 6575 2491 60  0000 C CNN
-F 2 "CustomFP:BQ21040" H 6450 2150 60  0001 C CNN
-F 3 "" H 6450 2150 60  0001 C CNN
-	1    6550 2200
-	1    0    0    -1
-$EndComp
-Connection ~ 6150 2050
-Connection ~ 7000 2050
-Wire Wire Line
-	8850 3650 9550 3650
-$Comp
 L Device:R R17
 U 1 1 5BB9C2E6
@@
 L Device:LED D5
 U 1 1 5BBA4754
-P 7450 2150
-F 0 "D5" H 7300 2000 50  0000 C CNN
-F 1 "LED" H 7450 2050 50  0000 C CNN
-F 2 "LEDs:LED_0805" H 7450 2150 50  0001 C CNN
-F 3 "~" H 7450 2150 50  0001 C CNN
-	1    7450 2150
+P 7400 2250
+F 0 "D5" H 7250 2100 50  0000 C CNN
+F 1 "LED" H 7400 2150 50  0000 C CNN
+F 2 "LEDs:LED_0805" H 7400 2250 50  0001 C CNN
+F 3 "~" H 7400 2250 50  0001 C CNN
+	1    7400 2250
 	1    0    0    -1
 $EndComp
@@
 L Device:R R13
 U 1 1 5BBA484E
-P 7750 2150
-F 0 "R13" V 7850 2150 50  0000 C CNN
-F 1 "330" V 7750 2150 50  0000 C CNN
-F 2 "Resistors_SMD:R_0805" V 7680 2150 50  0001 C CNN
-F 3 "~" H 7750 2150 50  0001 C CNN
-	1    7750 2150
+P 7700 2250
+F 0 "R13" V 7800 2250 50  0000 C CNN
+F 1 "330" V 7700 2250 50  0000 C CNN
+F 2 "Resistors_SMD:R_0805" V 7630 2250 50  0001 C CNN
+F 3 "~" H 7700 2250 50  0001 C CNN
+	1    7700 2250
 	0    1    1    0
 $EndComp
 $Comp
-L Device:Thermistor_NTC TH2
-U 1 1 5BBA528E
-P 8850 4100
-F 0 "TH2" H 8947 4146 50  0000 L CNN
-F 1 "NTC" H 8947 4055 50  0000 L CNN
-F 2 "Resistors_SMD:R_0805" H 8850 4150 50  0001 C CNN
-F 3 "~" H 8850 4150 50  0001 C CNN
-	1    8850 4100
-	1    0    0    -1
-$EndComp
-$Comp
 L Device:R R9
 U 1 1 5BBA53D0
 P 6000 2300
 F 0 "R9" H 6150 2250 50  0000 R CNN
-F 1 "Riset" H 6250 2350 50  0000 R CNN
+F 1 "1k" H 6250 2350 50  0000 R CNN
 F 2 "Resistors_SMD:R_0805" V 5930 2300 50  0001 C CNN
 F 3 "~" H 6000 2300 50  0001 C CNN
@@
 L Device:R R10
 U 1 1 5BBA5B49
-P 7300 3450
-F 0 "R10" H 7150 3500 50  0000 L CNN
-F 1 "100" H 7100 3400 50  0000 L CNN
-F 2 "Resistors_SMD:R_0805" V 7230 3450 50  0001 C CNN
-F 3 "~" H 7300 3450 50  0001 C CNN
-	1    7300 3450
+P 7200 3300
+F 0 "R10" H 7250 3400 50  0000 L CNN
+F 1 "100" V 7200 3250 50  0000 L CNN
+F 2 "Resistors_SMD:R_0805" V 7130 3300 50  0001 C CNN
+F 3 "~" H 7200 3300 50  0001 C CNN
+	1    7200 3300
 	1    0    0    -1
 $EndComp
@@
 L Device:R R12
 U 1 1 5BBA5CD3
-P 7600 3450
-F 0 "R12" H 7650 3500 50  0000 L CNN
-F 1 "100" H 7650 3400 50  0000 L CNN
-F 2 "Resistors_SMD:R_0805" V 7530 3450 50  0001 C CNN
-F 3 "~" H 7600 3450 50  0001 C CNN
-	1    7600 3450
+P 7700 3300
+F 0 "R12" H 7750 3450 50  0000 L CNN
+F 1 "100" V 7700 3250 50  0000 L CNN
+F 2 "Resistors_SMD:R_0805" V 7630 3300 50  0001 C CNN
+F 3 "~" H 7700 3300 50  0001 C CNN
+	1    7700 3300
 	1    0    0    -1
 $EndComp
@@
 L Device:C C3
 U 1 1 5BBA5DE1
-P 7450 3300
-F 0 "C3" V 7198 3300 50  0000 C CNN
-F 1 "0.1u" V 7289 3300 50  0000 C CNN
-F 2 "Capacitors_SMD:C_0805" H 7488 3150 50  0001 C CNN
-F 3 "~" H 7450 3300 50  0001 C CNN
-	1    7450 3300
+P 7450 3150
+F 0 "C3" V 7198 3150 50  0000 C CNN
+F 1 "0.1u" V 7289 3150 50  0000 C CNN
+F 2 "Capacitors_SMD:C_0805" H 7488 3000 50  0001 C CNN
+F 3 "~" H 7450 3150 50  0001 C CNN
+	1    7450 3150
 	0    1    1    0
 $EndComp
-Connection ~ 7300 3300
-Connection ~ 7600 3300
 $Comp
 L Device:Thermistor_NTC TH1
 U 1 1 5BBA73DD
-P 7100 2550
-F 0 "TH1" H 7197 2596 50  0000 L CNN
-F 1 "NTC" H 7197 2505 50  0000 L CNN
-F 2 "Resistors_SMD:R_0805" H 7100 2600 50  0001 C CNN
-F 3 "~" H 7100 2600 50  0001 C CNN
-	1    7100 2550
-	1    0    0    -1
+P 7050 2600
+F 0 "TH1" H 6800 2650 50  0000 L CNN
+F 1 "NTC" H 6800 2600 50  0000 L CNN
+F 2 "Resistors_SMD:R_0805" H 7050 2650 50  0001 C CNN
+F 3 "~" H 7050 2650 50  0001 C CNN
+	1    7050 2600
+	-1   0    0    1
 $EndComp
 Wire Wire Line
-	7000 2050 7900 2050
-Wire Wire Line
 	10800 2050 10800 2150
 Wire Wire Line
@@
 Wire Wire Line
 	8200 3300 8200 4250
-Wire Wire Line
-	7900 2150 7900 2050
 Connection ~ 7900 2050
 Wire Wire Line
@@
 	10600 3200 10600 3650
 Wire Wire Line
-	10600 3100 10500 3100
-Wire Wire Line
-	10500 3100 10500 3850
+	7950 3200 8350 3200
 $Comp
-L Device:Jumper_NO_Small JP4
-U 1 1 5BF51354
-P 8750 3950
-F 0 "JP4" H 8750 4135 50  0000 C CNN
-F 1 "Jumper_NO_Small" H 8750 4044 50  0000 C CNN
-F 2 "Jumpers:SMT-JUMPER_2_NO_NO-SILK" H 8750 3950 50  0001 C CNN
-F 3 "~" H 8750 3950 50  0001 C CNN
-	1    8750 3950
+L CustomComponents:R_0612 R98
+U 1 1 5BF27423
+P 7450 3550
+F 0 "R98" H 7450 3450 50  0000 C CNN
+F 1 "R_0612" H 7450 3750 50  0000 C CNN
+F 2 "Resistor_SMD:R_Shunt_Vishay_WSKW0612" H 7450 3550 50  0001 C CNN
+F 3 "" H 7450 3550 50  0001 C CNN
+	1    7450 3550
+	1    0    0    1
+$EndComp
+Connection ~ 8150 3650
+NoConn ~ 10600 3100
+$Comp
+L Device:Thermistor_NTC TH2
+U 1 1 5BBA528E
+P 7950 3400
+F 0 "TH2" H 8047 3446 50  0000 L CNN
+F 1 "NTC" H 8047 3355 50  0000 L CNN
+F 2 "Resistors_SMD:R_0805" H 7950 3450 50  0001 C CNN
+F 3 "~" H 7950 3450 50  0001 C CNN
+	1    7950 3400
 	1    0    0    -1
 $EndComp
 Wire Wire Line
-	8850 4250 9550 4250
+	8850 3650 10200 3650
 Wire Wire Line
-	9550 4250 9550 3650
-Connection ~ 9550 3650
+	7950 3200 7950 3250
 Wire Wire Line
-	9550 3650 10200 3650
-$Comp
-L Device:Jumper_NO_Small JP3
-U 1 1 5BF52D7D
-P 8750 3850
-F 0 "JP3" H 8750 4035 50  0000 C CNN
-F 1 "Jumper_NO_Small" H 8750 3944 50  0000 C CNN
-F 2 "Jumpers:SMT-JUMPER_2_NO_NO-SILK" H 8750 3850 50  0001 C CNN
-F 3 "~" H 8750 3850 50  0001 C CNN
-	1    8750 3850
-	1    0    0    -1
-$EndComp
+	7950 3550 7950 3650
+Connection ~ 7950 3650
 Wire Wire Line
-	8850 3850 10500 3850
+	7950 3650 8150 3650
 Wire Wire Line
-	8650 3850 8650 3950
+	7200 3000 7200 3150
 Wire Wire Line
-	8650 3850 7950 3850
+	7300 3150 7200 3150
+Connection ~ 7200 3150
 Wire Wire Line
-	7950 3850 7950 3200
+	7600 3150 7700 3150
 Wire Wire Line
-	7950 3200 8350 3200
-Connection ~ 8650 3850
-$Comp
-L CustomComponents:R_0612 U9
-U 1 1 5BF27423
-P 7450 3700
-F 0 "U9" H 7450 3485 50  0000 C CNN
-F 1 "R_0612" H 7450 3576 50  0000 C CNN
-F 2 "Resistor_SMD:R_Shunt_Vishay_WSKW0612" H 7450 3700 50  0001 C CNN
-F 3 "" H 7450 3700 50  0001 C CNN
-	1    7450 3700
-	1    0    0    1
-$EndComp
+	7700 3150 7700 3100
+Connection ~ 7700 3150
 Wire Wire Line
-	7200 3700 7200 3600
+	7700 3450 7700 3550
 Wire Wire Line
-	7200 3600 7300 3600
+	7200 3450 7200 3550
 Wire Wire Line
-	7600 3600 7700 3600
+	7700 3650 7950 3650
 Wire Wire Line
-	7700 3600 7700 3700
+	6150 3650 7050 3650
 Wire Wire Line
-	7700 3800 7850 3800
+	7000 2250 7250 2250
 Wire Wire Line
-	7850 3800 7850 3650
+	7850 2250 7900 2250
 Wire Wire Line
-	7850 3650 8150 3650
-Connection ~ 8150 3650
+	7900 2050 7900 2250
+Wire Wire Line
+	7000 2050 7900 2050
+Wire Wire Line
+	7050 2150 7000 2150
 Wire Wire Line
-	7200 3800 7100 3800
+	7050 2150 7050 2450
 Wire Wire Line
-	7100 3800 7100 3650
-Connection ~ 7100 3650
+	7050 2750 7050 3650
+Connection ~ 7050 3650
+Wire Wire Line
+	7050 3650 7200 3650
+$Comp
+L CustomComponents:BQ21040 U?
+U 1 1 5C00504B
+P 6550 2200
+F 0 "U?" H 6575 2597 60  0000 C CNN
+F 1 "BQ21040" H 6575 2491 60  0000 C CNN
+F 2 "" H 6450 2150 60  0001 C CNN
+F 3 "" H 6450 2150 60  0001 C CNN
+	1    6550 2200
+	1    0    0    -1
+$EndComp
+Connection ~ 6150 2050
+Connection ~ 7000 2050
 $EndSCHEMATC
