File: DoorUnlocker/RPI_zeroW_reset/RPI_zeroW_reset.sch (KiCad schematic (older format))
At the start: 4 parts, among them J1 Conn_01x02, SW1 Button, U1 TPL5111

Commit message: pcb updates
Parts:
- removed J1: Conn_01x02, CustomFP:PinHeader_1x02_P2.54mm_Horizontal, symbol CustomComponents:Conn_01x02
- removed SW1: Button, EbayParts:Tact_SMD_Switch, symbol JS_ElectroMechanical:Button
- added C1: C_Small, Capacitors:0805, symbol Device:C_Small
- added J1: RPI_Conn, Connector_PinHeader_2.54mm:PinHeader_2x02_P2.54mm_Vertical, symbol Connector_Generic:Conn_02x02_Top_Bottom
- added J2: Conn_01x01, Connector_PinHeader_2.54mm:PinHeader_1x01_P2.54mm_Vertical, symbol CustomComponents:Conn_01x01
- added Q1: BSS83P, Silicon-Standard:SOT323, symbol Transistor_FET:BSS83P
- added R2: R, Resistor_SMD:R_0805_2012Metric, symbol Device:R
- added RV1: R_POT, CustomFP:Bourns_TC33X-2, symbol Device:R_POT
- added SW1: SW_Push, EbayParts:Tact_SMD_Switch, symbol Switch:SW_Push
- added SW2: SW_SPST, CustomFP:SWITCH_SPDT_PTH, symbol Switch:SW_SPST
- R1: footprint Resistors:1206 -> Resistor_SMD:R_0805_2012Metric
- U1: footprint kicad-open-modules:SOT-23-6 -> Package_TO_SOT_SMD:SOT-23-6
Connections:
- net +5V: now reaches U1.1 (Vdd), U1.6 (EN/SHOT)
- net +5V: now also R1.2, C1.2, SW1.2, SW2.2 (B); no longer U1.5 (DRVn)
- net at R1.1: now also U1.5 (DRVn), Q1.1 (G); no longer U1.2 (GND)
- net at U1.3 (Delay): now also RV1.1, SW1.1; no longer R1.2
- net GPIO26: now reaches U1.4 (DONE)
- net GPIO26: now also J1.1 (Pin_1), R2.2
- new net: J2.1 (Pin_1), SW2.1 (A)
- new net GND: C1.1, J1.2 (Pin_2), J1.3 (Pin_3), Q1.3 (D), R2.1, RV1.2, U1.2 (GND)
- new net RUN: J1.4 (Pin_4), Q1.2 (S)
