File: PowerSupply/PowerSupply/PowerSupply - Copy.sch (KiCad schematic (older format))
At the start: 33 parts

Commit message: pcb updates
Parts:
- removed J?: touchLCD, symbol CustomComponents:touchLCD
- removed R?: Rsense, symbol Device:R
- added F1, F2, F3: Polyfuse, Fuse:Fuse_1206_3216Metric, symbol Device:Polyfuse
- added H1: 5V_load, TestPoint:TestPoint_Pad_D2.5mm, symbol Mechanical:MountingHole_Pad
- added H2: 5V_load_GND, TestPoint:TestPoint_Pad_D2.5mm, symbol Mechanical:MountingHole_Pad
- added H3: 5V_USB, TestPoint:TestPoint_Pad_D2.5mm, symbol Mechanical:MountingHole_Pad
- added H4: 5V_OUT, MountingHole:MountingHole_2.2mm_M2_Pad_Via, symbol Mechanical:MountingHole_Pad
- added H5: 12V_OUT, MountingHole:MountingHole_2.2mm_M2_Pad_Via, symbol Mechanical:MountingHole_Pad
- added H6: 3p3V_OUT, MountingHole:MountingHole_2.2mm_M2_Pad_Via, symbol Mechanical:MountingHole_Pad
- added H7: GND_OUT, MountingHole:MountingHole_2.2mm_M2_Pad_Via, symbol Mechanical:MountingHole_Pad
- added J1: Conn_01x04_Female, Connectors2:1X04, symbol Connector:Conn_01x04_Female
- added J2: ATX24, CustomFP:ATX_PWR_25pin, symbol atx24:ATX24
- added J3: PS_ON, Connectors2:1X02, symbol Connector:Conn_01x02_Female
- added R14, R15: R, Resistors_SMD:R_0805, symbol Device:R
- added U6: R_0612, Resistor_SMD:R_Shunt_Vishay_WSKW0612, symbol CustomComponents:R_0612
- added U?: ATmega328P-AU, Package_QFP:TQFP-32_7x7mm_P0.8mm, symbol MCU_Microchip_ATmega:ATmega328P-AU
- A1: renamed from A?; footprint Module:Arduino_Nano -> CustomPS:arduino_nano
- C1, C2, C3, C4: renamed from C?; footprint (none) -> Capacitors:0805
- P1: renamed from P?; footprint (none) -> CustomPS:uMAX-uSOP_10
- Q1: renamed from Q?; footprint (none) -> SMD_Packages:SO-8_PowerPAK_Vishay_Single
- Q2, Q3, Q4: renamed from Q?; footprint (none) -> kicad-open-modules:PowerPAK-1212-8
- Q5, Q6, Q7, Q8: renamed from Q?; footprint Package_TO_SOT_SMD:SOT-23 -> SMD_Packages_oj:SOT23
- R1, R10, R11, R12, R13, R2, R3, R4, R5, R6, R7, R9: renamed from R?; footprint (none) -> Resistors_SMD:R_0805
- U1, U2, U3: renamed from U?; value ACS70331EESATR-005U3 -> ACS70331; footprint ALLEGRO_ACS70331EESATR-005U3 -> ACS70331EESATR-005U3:ALLEGRO_ACS70331EESATR-005U3
- U4: renamed from U?; footprint 21-0140L_T2855-3 -> CustomFP:MAX11136ATI&plus_
- U5: renamed from U?; footprint 21-0036K -> CustomFP:MAX6126B30&plus_
Connections:
- net 5V_DIV_Out is gone; now on net 5V_DIV_OUT: R1.2, R2.1
- net SPI_LCD_CS_PINX is gone; now on net SPI_ADC_CS_PINX: A1.13 (D10)
- net +12V: now also F3.1, J2.10 (12V), J2.11 (12V); no longer U3.1 (IP+), U3.2 (IP+)
- net +3V3: now also A1.30 (VIN), F1.1, J1.4 (Pin_4), J2.1 (3V3), J2.12 (3V3), J2.13 (3V3), J2.2 (3V3); no longer P1.5 (INA+), U1.1 (IP+), U1.2 (IP+)
- net 12V_EN: now also A1.8 (D5)
- net 12V_Out: now also H5.1
- net 3V3_COURSE_EN: now also A1.10 (D7)
- net 3V3_FINE_EN: now also A1.11 (D8)
- net 3V3_Out: now also H6.1
- net 5V_DIV_OUT: now also U4.2 (AIN4); no longer U4.1 (AIN3)
- net 5V_EN: now also A1.9 (D6)
- net 5V_Out: now also H4.1
- net CNVST_PINX: now also A1.7 (D4); no longer A1.9 (D6)
- net EOC_PINX: now also A1.6 (D3); no longer A1.10 (D7)
- net GND: now also H2.1, H7.1, J1.3 (Pin_3), J2.15 (GND), J2.19 (GND), J2.7 (GND), R14.2; no longer A1.29 (GND)
- net SPI_3V3_CS_PINX: now also A1.12 (D9); no longer A1.11 (D8)
- net SPI_ADC_CS_PINX: no longer A1.12 (D9)
- net at A1.1 (D1/TX): now also J1.1 (Pin_1)
- net POK: now reaches A1.19 (A0)
- net POK: now also R14.1, R15.1
- net at A1.2 (D0/RX): now also J1.2 (Pin_2)
- net 3.3VA_D2: now reaches Q3.3 (Drain), U1.3 (IP-), U1.4 (IP-)
- net at U2.10 (VIOUT): now also U4.4 (AIN6); no longer U4.2 (AIN4)
- net at U4.27 (AIN1): no longer P1.8 (OUTA)
- net at U3.10 (VIOUT): now also U4.5 (AIN7); no longer U4.4 (AIN6)
- net at P1.4 (INA-): now also U6.2 (S-); no longer Q2.3 (Drain)
- net 5VA_D: now reaches Q4.3 (Drain), U2.3 (IP-), U2.4 (IP-)
- net 12VA_S: now reaches Q1.1 (Source), Q1.2 (Source), Q1.3 (Source), U3.3 (IP-), U3.4 (IP-)
- net +5V renamed 5V_A
- net 5V_A: now also F2.2
- new net: P1.5 (INA+), U6.3 (S+)
- new net: J2.16 (PS_ON), J3.1 (Pin_1)
- new net: J2.17 (GND), J3.2 (Pin_2)
- new net: H1.1, J2.21 (5V)
- new net: J2.8 (POK), R15.2
- new net: U?.21 (GND), U?.3 (GND), U?.5 (GND)
- new net: U?.4 (VCC), U?.6 (VCC)
- new net 12V_A: F3.2, U3.1 (IP+), U3.2 (IP+)
- new net 3.3VA_D1: Q2.3 (Drain), U6.4 (P-)
- new net 3.3V_A: F1.2, U1.1 (IP+), U1.2 (IP+), U6.1 (P+)
- new net 3V3_Fine_Out: P1.8 (OUTA), U4.1 (AIN3)
- new net 5VA: F2.1, J2.4 (5V), J2.6 (5V)
- new net 5V_USB: H3.1, J2.9 (5VSB)
- no-connect marks 3 -> 23
Other:
- moved on the sheet: A1
