File: WeatherStation/weatherStation/BMS.sch (KiCad schematic (older format))
At the start: 31 parts, among them J2 Conn_01x03, J5 Conn_01x02, J6 Conn_01x04, Q1 AO4430, SW2 SW_SPDT, U10 MAX40200, U11 MAX17048, U12 LM3671, U13 BQ24210, U8 BQ297xy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

Commit message: commit before more
Parts:
- removed C14: 4.7uF, Capacitor_SMD:C_0805_2012Metric, symbol Device:C_Small
- removed C15: 10uF, Capacitor_SMD:C_0805_2012Metric, symbol Device:C_Small
- removed D4, D5: LED, LED_SMD:LED_0805_2012Metric, symbol Device:LED
- removed D6, D7: D_Schottky, Diode_SMD:D_SOD-323, symbol Device:D_Schottky
- removed J6: Conn_01x04, Connector_JST:JST_GH_SM06B-GHS-TB_1x06-1MP_P1.25mm_Horizontal, symbol Connector_Generic:Conn_01x04
- removed L1: 2.2uH, Inductor_SMD:L_0805_2012Metric, symbol pspice:INDUCTOR
- removed Q1: AO4430, Package_SO:SOIC-8_3.9x4.9mm_P1.27mm, symbol CustomComponents:AO4430
- removed R16, R6, R8: 330, Resistor_SMD:R_0805_2012Metric, symbol Device:R_Small_US
- removed R7: 2.2k, Resistor_SMD:R_0805_2012Metric, symbol Device:R_Small_US
- removed U10: MAX40200, Package_TO_SOT_SMD:SOT-23-5, symbol CustomComponents:MAX40200
- removed U12: LM3671, Package_TO_SOT_SMD:SOT-23-5, symbol CustomComponents:LM3671
- removed U8: BQ297xy, Package_SON:WSON-6_1.5x1.5mm_P0.5mm, symbol Battery_Management:BQ297xy
- removed U9: ECH8693R, CustomFP:sot-28, symbol CustomComponents:ECH8693R
- removed W1, W3: Wire_Jump, CustomFP:wireJump, symbol CustomComponents:Wire_Jump
- added J3: Conn_01x02_Female, Connector_PinHeader_2.54mm:PinHeader_1x02_P2.54mm_Vertical, symbol Connector:Conn_01x02_Female
- added JP4, JP5: J_NO, Jumpers:SMT-JUMPER_2_NO_NO-SILK, symbol Device:Jumper_NO_Small
- added NT1, NT2, NT3, NT4: Net-Tie_2, NetTie:NetTie-2_SMD_Pad0.5mm, symbol Device:Net-Tie_2
- added R1: 10k, Resistor_SMD:R_0603_1608Metric, symbol Device:R_Small_US
- C16, C2: value 0.1uF -> 1uF
- J2: footprint CustomFP:JST_EH_B03B-EH-A_1x03_P1.50mm_Vertical -> Connector_JST:JST_PH_B3B-PH-K_1x03_P2.00mm_Vertical
- R10, R12: footprint Resistor_SMD:R_0805_2012Metric -> Resistor_SMD:R_0603_1608Metric
- R11: value 330 -> 750; footprint Resistor_SMD:R_0805_2012Metric -> Resistor_SMD:R_0603_1608Metric
- R9: value 330 -> 100k; footprint Resistor_SMD:R_0805_2012Metric -> Resistor_SMD:R_0603_1608Metric
- U11: footprint Package_DFN_QFN:TDFN-8-1EP_3x2mm_P0.5mm_EP1.80x1.65mm -> CustomFP:TQFN-8_2x2x0.75
Connections:
- net Batt- is gone; now on net GND: C2.2, J2.1 (Pin_1)
- net Pack- is gone; now on net GND: C16.2, C9.1, J5.2 (Pin_2), R11.2, R12.2, U11.1 (CTG), U11.4 (GND), U11.6 (QSTRT), U11.9 (GND), U13.3 (VSS)
- net Batt+: now also C2.1, J3.2 (Pin_2), NT1.1, NT2.1; no longer C9.2, R9.1, U11.2 (CELL), U11.3 (VDD), U13.10 (BAT)
- net GND: now also J3.1 (Pin_1), NT3.1, NT3.2, NT4.1, NT4.2
- net NTC: now also R10.2, U13.5 (TS); no longer R10.1, U13.7 (~EN)
- net at U13.4 (VTSB): now also R10.1
- net at U13.6 (~PG): now also R9.2, R1.1
- net at U13.8 (~CHG): now also JP4.2
- net Batt_int: now reaches J2.3 (Pin_3), SW2.2 (B)
- new net: JP5.2, R1.2, U13.7 (~EN)
- new net BattMon+: C9.2, NT1.2, U11.2 (CELL), U11.3 (VDD)
- new net Batt_Chrg+: JP4.1, NT2.2, R9.1, U13.10 (BAT)
- new net CHRG_EN: JP5.1
- no-connect marks 2 -> 1
Other:
- note removed: "Fixed DC-DC, 3.3V"
- note removed: "Power Switch"
- note removed: "Tx/Rx relative to uC"
- moved on the sheet: C9, J5, R10, R9
